Commit message: fixing urdf

File: server/static/RON/urdf/RON.urdf (robot description, URDF)
Before this commit: robot RON, 7 links, 6 joints
Joints:
- joint arm_left_joint_1: limit lower=0 upper=0 effort=0 velocity=0 -> lower=-3.1416 upper=3.1416 effort=0 velocity=0
- joint arm_left_joint_2: limit lower=0 upper=0 effort=0 velocity=0 -> lower=-3.1416 upper=3.1416 effort=0 velocity=0
- joint arm_right_joint_1: limit lower=0 upper=0 effort=0 velocity=0 -> lower=-3.1416 upper=3.1416 effort=0 velocity=0
- joint arm_right_joint_2: limit lower=0 upper=0 effort=0 velocity=0 -> lower=-3.1416 upper=3.1416 effort=0 velocity=0
